Commit message: added first attempt for ad astra URDF models and meshes

File: urdf/ad_astra.urdf (robot description, URDF)
Before this commit: robot ad_astra, 0 links, 0 joints
Links:
- added link rover, mass 44.9551052086405; collision mesh filename=package://New Rover 2.08 12.18.18 URDF and Meshes/meshes/ro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; visual mesh filename=package://New Rover 2.08 12.18.18 URDF and Meshes/meshes/ro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

Commit message: changed ad_astra URDF model and meshes over to my 2nd attempt

File: urdf/ad_astra.urdf (robot description, URDF)
Before this commit: robot New Rover 2.08 12.18.18 URDF and Meshes, 1 links, 0 joints
Links:
- added link arm_link1, mass 0.720067118020386; collision mesh filename=package://New Rover 2.08 12.18.18.SLDASM/meshes/arm_link1.S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; visual mesh filename=package://New Rover 2.08 12.18.18.SLDASM/meshes/arm_link1.S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
- added link arm_link2, mass 2.23804464644257; collision mesh filename=package://New Rover 2.08 12.18.18.SLDASM/meshes/arm_link2.S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; visual mesh filename=package://New Rover 2.08 12.18.18.SLDASM/meshes/arm_link2.S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
- added link arm_link3, mass 0.203954106945647; collision mesh filename=package://New Rover 2.08 12.18.18.SLDASM/meshes/arm_link3.S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; visual mesh filename=package://New Rover 2.08 12.18.18.SLDASM/meshes/arm_link3.S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
- added link chassis_link, mass 9.14786758671654; collision mesh filename=package://New Rover 2.08 12.18.18.SLDASM/meshes/chassis_lin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; visual mesh filename=package://New Rover 2.08 12.18.18.SLDASM/meshes/chassis_lin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
- added link left_train_link1, mass 3.60174015051005; collision mesh filename=package://New Rover 2.08 12.18.18.SLDASM/meshes/left_train_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; visual mesh filename=package://New Rover 2.08 12.18.18.SLDASM/meshes/left_train_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
- added link left_train_link2, mass 6.33331269612713; collision mesh filename=package://New Rover 2.08 12.18.18.SLDASM/meshes/left_train_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; visual mesh filename=package://New Rover 2.08 12.18.18.SLDASM/meshes/left_train_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
- added link right_train_link1, mass 3.69689838790142; collision mesh filename=package://New Rover 2.08 12.18.18.SLDASM/meshes/right_train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; visual mesh filename=package://New Rover 2.08 12.18.18.SLDASM/meshes/right_train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
- added link right_train_link2, mass 6.3263143064534; collision mesh filename=package://New Rover 2.08 12.18.18.SLDASM/meshes/right_train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; visual mesh filename=package://New Rover 2.08 12.18.18.SLDASM/meshes/right_train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
- link rover: mass 44.9551052086405 -> 35.8886782840091; geometry collision mesh filename=package://New Rover 2.08 12.18.18.SLDASM/meshes/rover.STL; visual mesh filename=package://New Rover 2.08 12.18.18.SLDASM/meshes/rover.STL
Joints:
- added joint arm_joint1: type revolute, parent rover, child arm_link1, origin xyz=0.51493 0.33908 -1.8382 rpy=0 0.87482 -3.091, axis 0 0 0, limit lower=0 upper=0 effort=0 velocity=0
- added joint arm_joint2: type revolute, parent rover, child arm_link2, origin xyz=0.55351 0.43414 -1.5311 rpy=-1.5708 0.0077357 -3.091, axis 0 0 0, limit lower=0 upper=0 effort=0 velocity=0
- added joint arm_joint3: type continuous, parent rover, child arm_link3, origin xyz=0.54402 0.34873 -1.382 rpy=-1.5708 -0.0077357 0.050544, axis 0 0 0
- added joint chassis_joint: type fixed, parent rover, child chassis_link, origin xyz=0.68321 0.60762 -1.2069 rpy=-1.5631 0 -1.4452, axis 0 0 0
- added joint left_train_joint1: type revolute, parent rover, child left_train_link1, origin xyz=0.63113 0.64768 -1.2613 rpy=0 -1.2217 -3.016, axis 0 0 0, limit lower=0 upper=0 effort=0 velocity=0
- added joint left_train_joint2: type revolute, parent rover, child left_train_link2, origin xyz=0.22048 0.53021 -0.9439 rpy=-1.5708 0.19992 -3.016, axis 0 0 0, limit lower=0 upper=0 effort=0 velocity=0
- added joint right_train_joint1: type revolute, parent rover, child right_train_link1, origin xyz=1.2304 0.15416 -1.0539 rpy=-1.6984 0 -1.4452, axis 0 0 0, limit lower=0 upper=0 effort=0 velocity=0
- added joint right_train_joint2: type revolute, parent rover, child right_train_link2, origin xyz=0.32989 -0.032815 -0.91339 rpy=-1.5708 0.020944 -3.016, axis 0 0 0, limit lower=0 upper=0 effort=0 velocity=0
